Commit message: Properly defined foot joints as fixed joints at the end of the legs; tuned GUI parameters for trotting

File: spotmicro/util/pybullet_data/FullAssemblyPyBullet/urdf/FullAssemblyPyBullet.urdf (robot description, URDF)
Before this commit: robot FullAssemblyPyBullet, 17 links, 16 joints
Links:
- removed link FL_Femur
- removed link FL_Hip
- removed link FL_Main
- removed link FL_Tibia
- removed link FR_Femur
- removed link FR_Hip
- removed link FR_Main
- removed link FR_Tibia
- removed link RL_Femur
- removed link RL_Hip
- removed link RL_Main
- removed link RL_Tibia
- removed link RR_Femur
- removed link RR_Hip
- removed link RR_Main
- removed link RR_Tibia
- added link FL_FemurLink, mass 0.162698622822929; collision mesh filename=package://FullAssemblyPyBullet/meshes/FL_FemurLink.STL; visual mesh filename=package://FullAssemblyPyBullet/meshes/FL_FemurLink.STL
- added link FL_FootLink, mass 0.00261710083689234; collision mesh filename=package://FullAssemblyPyBullet/meshes/FL_FootLink.STL; visual mesh filename=package://FullAssemblyPyBullet/meshes/FL_FootLink.STL
- added link FL_HipLink, mass 0.092628; collision mesh filename=package://FullAssemblyPyBullet/meshes/FL_HipLink.STL; visual mesh filename=package://FullAssemblyPyBullet/meshes/FL_HipLink.STL
- added link FL_TibiaLink, mass 0.109672208230102; collision mesh filename=package://FullAssemblyPyBullet/meshes/FL_TibiaLink.STL; visual mesh filename=package://FullAssemblyPyBullet/meshes/FL_TibiaLink.STL
- added link FR_FemurLink, mass 0.1627; collision mesh filename=package://FullAssemblyPyBullet/meshes/FR_FemurLink.STL; visual mesh filename=package://FullAssemblyPyBullet/meshes/FR_FemurLink.STL
- added link FR_FootLink, mass 0.0026171; collision mesh filename=package://FullAssemblyPyBullet/meshes/FR_FootLink.STL; visual mesh filename=package://FullAssemblyPyBullet/meshes/FR_FootLink.STL
- added link FR_HipLink, mass 0.092628; collision mesh filename=package://FullAssemblyPyBullet/meshes/FR_HipLink.STL; visual mesh filename=package://FullAssemblyPyBullet/meshes/FR_HipLink.STL
- added link FR_TibiaLink, mass 0.10967; collision mesh filename=package://FullAssemblyPyBullet/meshes/FR_TibiaLink.STL; visual mesh filename=package://FullAssemblyPyBullet/meshes/FR_TibiaLink.STL
- added link RL_FemurLink, mass 0.162698622211317; collision mesh filename=package://FullAssemblyPyBullet/meshes/RL_FemurLink.STL; visual mesh filename=package://FullAssemblyPyBullet/meshes/RL_FemurLink.STL
- added link RL_FootLink, mass 0.00261710083689218; collision mesh filename=package://FullAssemblyPyBullet/meshes/RL_FootLink.STL; visual mesh filename=package://FullAssemblyPyBullet/meshes/RL_FootLink.STL
- added link RL_HipLink, mass 0.0926275808970222; collision mesh filename=package://FullAssemblyPyBullet/meshes/RL_HipLink.STL; visual mesh filename=package://FullAssemblyPyBullet/meshes/RL_HipLink.STL
- added link RL_TibiaLink, mass 0.109672208230101; collision mesh filename=package://FullAssemblyPyBullet/meshes/RL_TibiaLink.STL; visual mesh filename=package://FullAssemblyPyBullet/meshes/RL_TibiaLink.STL
- added link RR_FemurLink, mass 0.16269859820821; collision mesh filename=package://FullAssemblyPyBullet/meshes/RR_FemurLink.STL; visual mesh filename=package://FullAssemblyPyBullet/meshes/RR_FemurLink.STL
- added link RR_FootLink, mass 0.00261710077329806; collision mesh filename=package://FullAssemblyPyBullet/meshes/RR_FootLink.STL; visual mesh filename=package://FullAssemblyPyBullet/meshes/RR_FootLink.STL
- added link RR_HipLink, mass 0.0926285030937892; collision mesh filename=package://FullAssemblyPyBullet/meshes/RR_HipLink.STL; visual mesh filename=package://FullAssemblyPyBullet/meshes/RR_HipLink.STL
- added link RR_TibiaLink, mass 0.109672400053178; collision mesh filename=package://FullAssemblyPyBullet/meshes/RR_TibiaLink.STL; visual mesh filename=package://FullAssemblyPyBullet/meshes/RR_TibiaLink.STL
- link MainBody: mass 1.62403957260971 -> 1.84238098815425
Joints:
- removed joint FL_Femur
- removed joint FL_Hip
- removed joint FL_Main
- removed joint FL_Tibia
- removed joint FR_Femur
- removed joint FR_Hip
- removed joint FR_Main
- removed joint FR_Tibia
- removed joint RL_Femur
- removed joint RL_Hip
- removed joint RL_Main
- removed joint RL_Tibia
- removed joint RR_Femur
- removed joint RR_Hip
- removed joint RR_Main
- removed joint RR_Tibia
- added joint FL_FemurJoint: type revolute, parent FL_HipLink, child FL_FemurLink, origin xyz=-0.054 -0.009 0 rpy=0 0 0, axis 0 1 0, limit lower=-0.785 upper=0.785 effort=0 velocity=0
- added joint FL_FootJoint: type fixed, parent FL_TibiaLink, child FL_FootLink, origin xyz=0.063753 0 -0.2336 rpy=0 0 0, axis 0 0 0
- added joint FL_HipJoint: type revolute, parent MainBody, child FL_HipLink, origin xyz=0.2878 0.1 0.037867 rpy=0 0 0, axis 1 0 0, limit lower=-0.175 upper=1.571 effort=0 velocity=0
- added joint FL_TibiaJoint: type revolute, parent FL_FemurLink, child FL_TibiaLink, origin xyz=-0.1283 0.0695 -0.1404 rpy=0 0 0, axis 0 1 0, limit lower=-1.571 upper=0 effort=0 velocity=0
- added joint FR_FemurJoint: type revolute, parent FR_HipLink, child FR_FemurLink, origin xyz=-0.054 0.009 0 rpy=0 0 0, axis 0 1 0, limit lower=-0.785 upper=0.785 effort=0 velocity=0
- added joint FR_FootJoint: type fixed, parent FR_TibiaLink, child FR_FootLink, origin xyz=0.0637534602692 0 -0.233603271727562 rpy=0 0 0, axis 0 0 0
- added joint FR_HipJoint: type revolute, parent MainBody, child FR_HipLink, origin xyz=0.2878 -0.1 0.037867 rpy=0 0 0, axis 1 0 0, limit lower=-1.571 upper=0.175 effort=0 velocity=0
- added joint FR_TibiaJoint: type revolute, parent FR_FemurLink, child FR_TibiaLink, origin xyz=-0.1283 -0.0695 -0.1404 rpy=0 0 0, axis 0 1 0, limit lower=-1.571 upper=0 effort=0 velocity=0
- added joint RL_FemurJoint: type revolute, parent RL_HipLink, child RL_FemurLink, origin xyz=-0.054 -0.009 0 rpy=0 0 0, axis 0 1 0, limit lower=-0.785 upper=0.785 effort=0 velocity=0
- added joint RL_FootJoint: type fixed, parent RL_TibiaLink, child RL_FootLink, origin xyz=0.0637534602692006 0 -0.233603271727562 rpy=0 0 0, axis 0 0 0
- added joint RL_HipJoint: type revolute, parent MainBody, child RL_HipLink, origin xyz=-0.1794 0.1 0.037 rpy=0 0 0, axis 1 0 0, limit lower=-0.175 upper=1.571 effort=0 velocity=0
- added joint RL_TibiaJoint: type revolute, parent RL_FemurLink, child RL_TibiaLink, origin xyz=-0.1283 0.0695 -0.1404 rpy=0 0 0, axis 0 1 0, limit lower=-1.571 upper=0 effort=0 velocity=0
- added joint RR_FemurJoint: type revolute, parent RR_HipLink, child RR_FemurLink, origin xyz=-0.054 0.009 0 rpy=0 0 0, axis 0 1 0, limit lower=-0.785 upper=0.785 effort=0 velocity=0
- added joint RR_FootJoint: type fixed, parent RR_TibiaLink, child RR_FootLink, origin xyz=0.0637534602692006 0 -0.233603271727562 rpy=0 0 0, axis 0 0 0
- added joint RR_HipJoint: type revolute, parent MainBody, child RR_HipLink, origin xyz=-0.1794 -0.1 0.037 rpy=0 0 0, axis 1 0 0, limit lower=-1.571 upper=0.175 effort=0 velocity=0
- added joint RR_TibiaJoint: type revolute, parent RR_FemurLink, child RR_TibiaLink, origin xyz=-0.1283 -0.0695 -0.1404 rpy=0 0 0, axis 0 1 0, limit lower=-1.571 upper=0 effort=0 velocity=0
