Commit message: imported spherically-shaped collision bodies for each of the feet

File: spotmicro/util/pybullet_data/FullAssemblyPyBullet/urdf/FullAssemblyCollisions.urdf (robot description, URDF)
Before this commit: robot FullAssemblyPyBullet, 17 links, 16 joints
Links:
- link FL_FootLink: geometry collision mesh filename=package://FullAssemblyPyBullet/meshes/FL_FootLinkCollision_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; visual mesh filename=package://FullAssemblyPyBullet/meshes/FL_FootLink.STL
- link FR_FootLink: geometry collision mesh filename=package://FullAssemblyPyBullet/meshes/FR_FootLinkCollision_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; visual mesh filename=package://FullAssemblyPyBullet/meshes/FR_FootLink.STL
- link RL_FootLink: geometry collision mesh filename=package://FullAssemblyPyBullet/meshes/RL_FootLinkCollision_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; visual mesh filename=package://FullAssemblyPyBullet/meshes/RL_FootLink.STL
- link RR_FootLink: geometry collision mesh filename=package://FullAssemblyPyBullet/meshes/RR_FootLinkCollision_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; visual mesh filename=package://FullAssemblyPyBullet/meshes/RR_FootLink.STL
